Commit message: first commit

File: assets/a2r_drone/urdf/a2r_drone.urdf (robot description, URDF)
Before this commit: robot a2r_drone, 5 links, 4 joints
Links:
- link prop1: geometry visual mesh filename=../meshes/propeller.obj scale=1 1 1
Joints:
- joint m1_joint: origin xyz=-0.122 -0.1343 0.013 rpy=0 0 0 -> xyz=-0.122 0.1343 0.013 rpy=0 0 0
- joint m2_joint: origin xyz=0.1482504096571687 -0.1047432515919767 0.013 rpy=0 0 0 -> xyz=0.1482504096571687 0.1047432515919767 0.013 rpy=0 0 0
- joint m3_joint: origin xyz=-0.122 0.1343 0.013 rpy=0 0 0 -> xyz=0.1482504096571687 -0.1047432515919767 0.013 rpy=0 0 0
- joint m4_joint: origin xyz=0.1482504096571687 0.1047432515919767 0.013 rpy=0 0 0 -> xyz=-0.122 -0.1343 0.013 rpy=0 0 0

Commit message: added xy bounds, changed dynamic parameters, antonio critica i miei commit

File: assets/a2r_drone/urdf/a2r_drone.urdf (robot description, URDF)
Before this commit: robot a2r_drone, 5 links, 4 joints
Joints:
- joint m1_joint: origin xyz=-0.122 0.1343 0.013 rpy=0 0 0 -> xyz=-0.122 -0.1343 0.013 rpy=0 0 0
- joint m2_joint: origin xyz=0.1482504096571687 0.1047432515919767 0.013 rpy=0 0 0 -> xyz=0.1482504096571687 -0.1047432515919767 0.013 rpy=0 0 0
- joint m3_joint: origin xyz=0.1482504096571687 -0.1047432515919767 0.013 rpy=0 0 0 -> xyz=-0.122 0.1343 0.013 rpy=0 0 0
- joint m4_joint: origin xyz=-0.122 -0.1343 0.013 rpy=0 0 0 -> xyz=0.1482504096571687 0.1047432515919767 0.013 rpy=0 0 0
